File: Hardware/Eagle Files/adns3050 v6.brd (EAGLE design)
At the start: 30.5 x 51.9 mm, 5 parts, among them U1 V_REG_317SMD

Commit message: Added components
Parts:
- added C2: (no value), rcl:R/2012-12R
- added C3: (no value), eagle-ltspice:C0603
Connections:
- net GND: now also C2.-, C3.2
- net VDD: now also C2.+, C3.1
Routing:
- net VDD: track 47.4 -> 53.2 mm
Other:
- board text added: "A1"
Changed lines of the file:
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@@
 <text x="18.415" y="-6.223" size="1.27" layer="21">M</text>
 <text x="20.447" y="-6.223" size="1.27" layer="21">NC</text>
+<text x="12.319" y="36.957" size="1.27" layer="21" rot="R180">A1</text>
 </plain>
 <attributes>
@@
 <attribute name="SPICEPREFIX" value="R" x="26.543" y="29.718" size="1.778" layer="27" display="off"/>
 </element>
-<element name="C1" library="eagle-ltspice" package="C0603" value="" x="9.271" y="30.607" rot="R90">
+<element name="C1" library="eagle-ltspice" package="C0603" value="" x="9.271" y="30.607" smashed="yes" rot="R90">
 <attribute name="SPICEMODEL" value="NONE" x="9.271" y="30.607" size="1.778" layer="27" rot="R90" display="off"/>
 <attribute name="SPICEPREFIX" value="C" x="9.271" y="30.607" size="1.778" layer="27" rot="R90" display="off"/>
+<attribute name="NAME" x="10.541" y="28.956" size="1.27" layer="25" rot="R180"/>
+<attribute name="VALUE" x="11.176" y="29.972" size="1.27" layer="27" rot="R90"/>
 </element>
 <element name="U$1" library="ADNS3050" package="ADNS3" value="3050" x="17.526" y="27.813" smashed="yes"/>
@@
 <attribute name="NAME" x="22.987" y="-0.127" size="1.27" layer="25" ratio="10" rot="R270"/>
 <attribute name="VALUE" x="22.733" y="2.413" size="1.27" layer="27" rot="R180"/>
+</element>
+<element name="C2" library="rcl" package="R/2012-12R" value="" x="7.874" y="9.652" smashed="yes">
+<attribute name="NAME" x="5.924" y="10.906" size="1.27" layer="25"/>
+<attribute name="VALUE" x="5.924" y="7.327" size="1.27" layer="27"/>
+</element>
+<element name="C3" library="eagle-ltspice" package="C0603" value="" x="7.112" y="30.607" smashed="yes" rot="R90">
+<attribute name="SPICEMODEL" value="NONE" x="7.112" y="30.607" size="1.778" layer="27" rot="R90" display="off"/>
+<attribute name="SPICEPREFIX" value="C" x="7.112" y="30.607" size="1.778" layer="27" rot="R90" display="off"/>
+<attribute name="NAME" x="8.255" y="28.956" size="1.27" layer="25" rot="R180"/>
+<attribute name="VALUE" x="9.017" y="29.972" size="1.27" layer="27" rot="R90"/>
 </element>
 </elements>
@@
 <contactref element="U1" pad="1"/>
 <via x="11.557" y="3.683" extent="1-16" drill="0.6" diameter="0.8128"/>
-<via x="6.731" y="31.496" extent="1-16" drill="0.6"/>
+<via x="7.112" y="33.401" extent="1-16" drill="0.6"/>
 <contactref element="JP1" pad="8"/>
+<contactref element="C2" pad="-"/>
+<contactref element="C3" pad="2"/>
 </signal>
 <signal name="VDD">
@@
 <wire x1="9.271" y1="29.757" x2="10.883" y2="29.757" width="0.4064" layer="1"/>
 <wire x1="10.883" y1="29.757" x2="11.176" y2="29.464" width="0.4064" layer="1"/>
-<wire x1="9.144" y1="6.4008" x2="9.144" y2="29.63" width="0.4064" layer="1"/>
 <wire x1="9.144" y1="29.63" x2="9.271" y2="29.757" width="0.4064" layer="1"/>
 <contactref element="JP1" pad="6"/>
@@
 <wire x1="17.653" y1="0.381" x2="17.653" y2="-2.032" width="0.4064" layer="1"/>
 <wire x1="17.653" y1="-2.032" x2="16.383" y2="-3.302" width="0.4064" layer="1"/>
+<contactref element="C2" pad="+"/>
+<contactref element="C3" pad="1"/>
+<wire x1="7.112" y1="29.757" x2="9.271" y2="29.757" width="0.4064" layer="1"/>
+<wire x1="9.144" y1="6.4008" x2="9.017" y2="6.4008" width="0.4064" layer="1"/>
+<wire x1="9.017" y1="6.4008" x2="9.017" y2="29.503" width="0.4064" layer="1"/>
+<wire x1="9.017" y1="29.503" x2="9.271" y2="29.757" width="0.4064" layer="1"/>
+<wire x1="9.049" y1="9.652" x2="9.049" y2="6.4958" width="0.4064" layer="1"/>
+<wire x1="9.049" y1="6.4958" x2="9.144" y2="6.4008" width="0.4064" layer="1"/>
 </signal>
 <signal name="MISO">
