File: Hardware/Eagle Files/adns3050 v6.sch (EAGLE design)
At the start: 5 parts, among them U1 V_REG_317SMD

Commit message: Added components
Parts:
- added C2: (no value), rcl:CPOL-EUR/2012-12R
- added C3: (no value), eagle-ltspice:CC0603
Connections:
- net GND: now also C2.-, C3.2
- net VDD: now also C2.+, C3.1
Changed lines of the file:
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@@
 <part name="SUPPLY7" library="supply2" deviceset="GND" device=""/>
 <part name="JP1" library="pinhead" deviceset="PINHD-2X4" device=""/>
+<part name="C2" library="rcl" deviceset="CPOL-EU" device="R/2012-12R"/>
+<part name="C3" library="eagle-ltspice" deviceset="C" device="C0603"/>
 </parts>
 <sheets>
@@
 <instance part="SUPPLY7" gate="GND" x="66.04" y="139.7"/>
 <instance part="JP1" gate="A" x="104.14" y="99.06"/>
+<instance part="C2" gate="G$1" x="63.5" y="114.3"/>
+<instance part="C3" gate="G$1" x="71.12" y="114.3"/>
 </instances>
 <busses>
@@
 <wire x1="76.2" y1="121.92" x2="81.28" y2="121.92" width="0.1524" layer="91"/>
 <label x="81.28" y="121.92" size="1.778" layer="95"/>
+<pinref part="C2" gate="G$1" pin="+"/>
+<wire x1="76.2" y1="116.84" x2="71.12" y2="116.84" width="0.1524" layer="91"/>
+<junction x="63.5" y="116.84"/>
+<pinref part="C3" gate="G$1" pin="1"/>
+<junction x="71.12" y="116.84"/>
+<wire x1="71.12" y1="116.84" x2="63.5" y2="116.84" width="0.1524" layer="91"/>
+<junction x="76.2" y="116.84"/>
 </segment>
 <segment>
@@
 <pinref part="C1" gate="G$1" pin="2"/>
 <pinref part="SUPPLY5" gate="GND" pin="GND"/>
+<pinref part="C2" gate="G$1" pin="-"/>
+<wire x1="63.5" y1="109.22" x2="71.12" y2="109.22" width="0.1524" layer="91"/>
+<junction x="76.2" y="109.22"/>
+<pinref part="C3" gate="G$1" pin="2"/>
+<junction x="71.12" y="109.22"/>
+<wire x1="71.12" y1="109.22" x2="76.2" y2="109.22" width="0.1524" layer="91"/>
+<junction x="63.5" y="109.22"/>
 </segment>
 <segment>
